Commit message: add new package for rviz2 and TF

File: src/patasmonkey_description/urdf/patasmonkey.urdf (robot description, URDF)
Before this commit: robot patasmonkey_v6, 11 links, 10 joints
Joints:
- joint rev7: child wheel_frontright -> wheel_rearright
- joint rev8: child wheel_rearright -> wheel_frontright

Commit message: add new package for rviz2 and TF

File: src/patasmonkey_description/urdf/patasmonkey.urdf (robot description, URDF)
Before this commit: robot patasmonkey_v6, 11 links, 10 joints
Links:
- removed link wheel_arm_frontright
- removed link wheel_arm_rearright
- removed link wheel_frontleft
- removed link wheel_frontright
- removed link wheel_rearleft
- removed link wheel_rearright
- added link frontleft_wheel_link, mass 0.6459736269326636; collision mesh filename=package://patasmonkey_description/meshes/wheel.stl scale=0.001 0.001 0.001; visual mesh filename=package://patasmonkey_description/meshes/wheel.stl scale=0.001 0.001 0.001
- added link frontright_wheel_link, mass 0.6459736269326636; collision mesh filename=package://patasmonkey_description/meshes/wheel.stl scale=0.001 0.001 0.001; visual mesh filename=package://patasmonkey_description/meshes/wheel.stl scale=0.001 0.001 0.001
- added link rearleft_wheel_link, mass 0.6459736269326636; collision mesh filename=package://patasmonkey_description/meshes/wheel.stl scale=0.001 0.001 0.001; visual mesh filename=package://patasmonkey_description/meshes/wheel.stl scale=0.001 0.001 0.001
- added link rearright_wheel_link, mass 0.6459736269326636; collision mesh filename=package://patasmonkey_description/meshes/wheel.stl scale=0.001 0.001 0.001; visual mesh filename=package://patasmonkey_description/meshes/wheel.stl scale=0.001 0.001 0.001
- added link wheel_arm_frontright_link, mass 0.06867212404052492; collision mesh filename=package://patasmonkey_description/meshes/wheel_arm.stl scale=0.001 0.001 0.001; visual mesh filename=package://patasmonkey_description/meshes/wheel_arm.stl scale=0.001 0.001 0.001
- added link wheel_arm_rearright_link, mass 0.06867212404052492; collision mesh filename=package://patasmonkey_description/meshes/wheel_arm.stl scale=0.001 0.001 0.001; visual mesh filename=package://patasmonkey_description/meshes/wheel_arm.stl scale=0.001 0.001 0.001
Joints:
- joint base_to_body_left: origin xyz=0 0 0 rpy=0 0 0  -> xyz=0 0 0 rpy=0 0 0
- joint rev3: child wheel_arm_frontright -> wheel_arm_rearright_link
- joint rev4: child wheel_arm_rearright -> wheel_arm_frontright_link
- joint rev5: child wheel_frontleft -> frontleft_wheel_link
- joint rev6: child wheel_rearleft -> rearleft_wheel_link
- joint rev7: child wheel_rearright -> rearright_wheel_link; parent wheel_arm_frontright -> wheel_arm_rearright_link
- joint rev8: child wheel_frontright -> frontright_wheel_link; parent wheel_arm_rearright -> wheel_arm_frontright_link

Commit message: update patasmonkey hardware structure

File: src/patasmonkey_description/urdf/patasmonkey.urdf (robot description, URDF)
Before this commit: robot patasmonkey_v6, 11 links, 10 joints
Links:
- removed link base_link
- removed link body_left_link
- removed link body_right_link
- removed link frontleft_wheel_link
- removed link frontright_wheel_link
- removed link rearleft_wheel_link
- removed link rearright_wheel_link
- removed link wheel_arm_frontleft_link
- removed link wheel_arm_frontright_link
- removed link wheel_arm_rearleft_link
- removed link wheel_arm_rearright_link
- added link base_link_v3:1, mass 8.831101767270535; collision mesh filename=package://patasmonkey_description/meshes/base_link.stl scale=0.001 0.001 0.001; visual mesh filename=package://patasmonkey_description/meshes/base_link.stl scale=0.001 0.001 0.001
- added link wheel_arm_v2:1, mass 0.06867212404052492; collision mesh filename=package://patasmonkey_description/meshes/wheel_arm.stl scale=0.001 0.001 0.001; visual mesh filename=package://patasmonkey_description/meshes/wheel_arm.stl scale=0.001 0.001 0.001
- added link wheel_arm_v2:2, mass 0.06867212404052492; collision mesh filename=package://patasmonkey_description/meshes/wheel_arm.stl scale=0.001 0.001 0.001; visual mesh filename=package://patasmonkey_description/meshes/wheel_arm.stl scale=0.001 0.001 0.001
- added link wheel_arm_v2:3, mass 0.06867212404052492; collision mesh filename=package://patasmonkey_description/meshes/wheel_arm.stl scale=0.001 0.001 0.001; visual mesh filename=package://patasmonkey_description/meshes/wheel_arm.stl scale=0.001 0.001 0.001
- added link wheel_arm_v2:4, mass 0.06867212404052492; collision mesh filename=package://patasmonkey_description/meshes/wheel_arm.stl scale=0.001 0.001 0.001; visual mesh filename=package://patasmonkey_description/meshes/wheel_arm.stl scale=0.001 0.001 0.001
- added link wheel_v2:1, mass 0.6459736269326636; collision mesh filename=package://patasmonkey_description/meshes/wheel.stl scale=0.001 0.001 0.001; visual mesh filename=package://patasmonkey_description/meshes/wheel.stl scale=0.001 0.001 0.001
- added link wheel_v2:2, mass 0.6459736269326636; collision mesh filename=package://patasmonkey_description/meshes/wheel.stl scale=0.001 0.001 0.001; visual mesh filename=package://patasmonkey_description/meshes/wheel.stl scale=0.001 0.001 0.001
- added link wheel_v2:3, mass 0.6459736269326636; collision mesh filename=package://patasmonkey_description/meshes/wheel.stl scale=0.001 0.001 0.001; visual mesh filename=package://patasmonkey_description/meshes/wheel.stl scale=0.001 0.001 0.001
- added link wheel_v2:4, mass 0.6459736269326636; collision mesh filename=package://patasmonkey_description/meshes/wheel.stl scale=0.001 0.001 0.001; visual mesh filename=package://patasmonkey_description/meshes/wheel.stl scale=0.001 0.001 0.001
Joints:
- removed joint base_to_body_left
- removed joint rev8
- joint rev0: axis 0.0 1.0 0.0 -> -1.0 0.0 0.0; child body_right_link -> wheel_arm_v2:1; origin xyz=0.0 0.01 0.06 rpy=0 0 0 -> xyz=0.09999999999999998 -0.03 0.03 rpy=0 0 0; parent body_left_link -> base_link_v3:1
- joint rev1: axis 0.0 1.0 0.0 -> -1.0 0.0 0.0; child wheel_arm_frontleft_link -> wheel_arm_v2:2; origin xyz=-0.029999999999999964 -0.15 0.029999999999999895 rpy=0 0 0 -> xyz=0.09999999999999998 0.03 0.03 rpy=0 0 0; parent body_left_link -> base_link_v3:1
- joint rev2: axis 0.0 1.0 0.0 -> 1.0 0.0 0.0; child wheel_arm_rearleft_link -> wheel_arm_v2:3; origin xyz=0.030000000000000054 -0.15 0.029999999999999992 rpy=0 0 0 -> xyz=-0.1 0.03 0.03 rpy=0 0 0; parent body_left_link -> base_link_v3:1
- joint rev3: axis 0.0 -1.0 0.0 -> 1.0 0.0 0.0; child wheel_arm_rearright_link -> wheel_arm_v2:4; origin xyz=0.02999999999999993 0.13999999999999996 -0.029999999999999954 rpy=0 0 0 -> xyz=-0.10000000000000002 -0.03 0.03 rpy=0 0 0; parent body_right_link -> base_link_v3:1
- joint rev4: axis 0.0 -1.0 0.0 -> 1.0 0.0 0.0; child wheel_arm_frontright_link -> wheel_v2:1; origin xyz=-0.03 0.13999999999999996 -0.029999999999999992 rpy=0 0 0 -> xyz=0.009999999999999981 -0.15035081932574534 -0.05472322293210702 rpy=0 0 0; parent body_right_link -> wheel_arm_v2:1
- joint rev5: axis 0.0 -0.9999999999999978 0.0 -> 1.0 0.0 0.0; child frontleft_wheel_link -> wheel_v2:2; origin xyz=-0.15035081932574496 -0.00999999999999987 -0.054723222932106956 rpy=0 0 0 -> xyz=0.010000000000000009 0.15035081932574534 -0.05472322293210699 rpy=0 0 0; parent wheel_arm_frontleft_link -> wheel_arm_v2:2
- joint rev6: axis 0.0 -0.9999999999999987 0.0 -> 1.0 0.0 0.0; child rearleft_wheel_link -> wheel_v2:3; origin xyz=0.15035081932574518 -0.00999999999999987 -0.05472322293210702 rpy=0 0 0 -> xyz=-0.009999999999999995 0.15035081932574534 -0.05472322293210699 rpy=0 0 0; parent wheel_arm_rearleft_link -> wheel_arm_v2:3
- joint rev7: axis 0.0 -0.9999999999999981 0.0 -> 1.0 0.0 0.0; child rearright_wheel_link -> wheel_v2:4; origin xyz=0.1503508193257454 0.009999999999999953 -0.05472322293210703 rpy=0 0 0 -> xyz=-0.010000000000000023 -0.15035081932574534 -0.05472322293210702 rpy=0 0 0; parent wheel_arm_rearright_link -> wheel_arm_v2:4

Commit message: update patasmonkey hardware structure

File: src/patasmonkey_description/urdf/patasmonkey.urdf (robot description, URDF)
Before this commit: robot patasmonkey_v2_v2, 9 links, 8 joints
Links:
- removed link base_link_v3:1
- removed link wheel_arm_v2:1
- removed link wheel_arm_v2:2
- removed link wheel_arm_v2:3
- removed link wheel_arm_v2:4
- added link base_link_v4:1, mass 8.831101767270535; collision mesh filename=package://patasmonkey_description/meshes/base_link.stl scale=0.001 0.001 0.001; visual mesh filename=package://patasmonkey_description/meshes/base_link.stl scale=0.001 0.001 0.001
- added link wheel_arm_v6:1, mass 0.34336062020263136; collision mesh filename=package://patasmonkey_description/meshes/wheel_arm.stl scale=0.001 0.001 0.001; visual mesh filename=package://patasmonkey_description/meshes/wheel_arm.stl scale=0.001 0.001 0.001
- added link wheel_arm_v6:2, mass 0.34336062020263136; collision mesh filename=package://patasmonkey_description/meshes/wheel_arm.stl scale=0.001 0.001 0.001; visual mesh filename=package://patasmonkey_description/meshes/wheel_arm.stl scale=0.001 0.001 0.001
- added link wheel_arm_v6:3, mass 0.34336062020263136; collision mesh filename=package://patasmonkey_description/meshes/wheel_arm.stl scale=0.001 0.001 0.001; visual mesh filename=package://patasmonkey_description/meshes/wheel_arm.stl scale=0.001 0.001 0.001
- added link wheel_arm_v6:4, mass 0.34336062020263136; collision mesh filename=package://patasmonkey_description/meshes/wheel_arm.stl scale=0.001 0.001 0.001; visual mesh filename=package://patasmonkey_description/meshes/wheel_arm.stl scale=0.001 0.001 0.001
Joints:
- joint rev0: child wheel_arm_v2:1 -> wheel_arm_v6:1; origin xyz=0.09999999999999998 -0.03 0.03 rpy=0 0 0 -> xyz=0.09999999999999998 -0.030000000000000006 0.05000000000000001 rpy=0 0 0; parent base_link_v3:1 -> base_link_v4:1
- joint rev1: child wheel_arm_v2:2 -> wheel_arm_v6:2; origin xyz=0.09999999999999998 0.03 0.03 rpy=0 0 0 -> xyz=0.09999999999999998 0.03 0.05 rpy=0 0 0; parent base_link_v3:1 -> base_link_v4:1
- joint rev2: child wheel_arm_v2:3 -> wheel_arm_v6:3; origin xyz=-0.1 0.03 0.03 rpy=0 0 0 -> xyz=-0.1 0.03 0.05 rpy=0 0 0; parent base_link_v3:1 -> base_link_v4:1
- joint rev3: child wheel_arm_v2:4 -> wheel_arm_v6:4; origin xyz=-0.10000000000000002 -0.03 0.03 rpy=0 0 0 -> xyz=-0.10000000000000002 -0.030000000000000006 0.05000000000000001 rpy=0 0 0; parent base_link_v3:1 -> base_link_v4:1
- joint rev4: origin xyz=0.009999999999999981 -0.15035081932574534 -0.05472322293210702 rpy=0 0 0 -> xyz=0.05000000000000002 -0.15035081932574534 -0.05472322293210703 rpy=0 0 0; parent wheel_arm_v2:1 -> wheel_arm_v6:1
- joint rev5: origin xyz=0.010000000000000009 0.15035081932574534 -0.05472322293210699 rpy=0 0 0 -> xyz=0.05000000000000002 0.15035081932574534 -0.054723222932107 rpy=0 0 0; parent wheel_arm_v2:2 -> wheel_arm_v6:2
- joint rev6: origin xyz=-0.009999999999999995 0.15035081932574534 -0.05472322293210699 rpy=0 0 0 -> xyz=-0.04999999999999999 0.15035081932574534 -0.054723222932107 rpy=0 0 0; parent wheel_arm_v2:3 -> wheel_arm_v6:3
- joint rev7: origin xyz=-0.010000000000000023 -0.15035081932574534 -0.05472322293210702 rpy=0 0 0 -> xyz=-0.05 -0.15035081932574534 -0.05472322293210703 rpy=0 0 0; parent wheel_arm_v2:4 -> wheel_arm_v6:4

Commit message: update link names

File: src/patasmonkey_description/urdf/patasmonkey.urdf (robot description, URDF)
Before this commit: robot patasmonkey_ugv, 9 links, 8 joints
Links:
- removed link base_link_v4:1
- removed link wheel_arm_v6:1
- removed link wheel_arm_v6:2
- removed link wheel_arm_v6:3
- removed link wheel_arm_v6:4
- removed link wheel_v2:1
- removed link wheel_v2:2
- removed link wheel_v2:3
- removed link wheel_v2:4
- added link base_link, mass 8.831101767270535; collision mesh filename=package://patasmonkey_description/meshes/base_link.stl scale=0.001 0.001 0.001; visual mesh filename=package://patasmonkey_description/meshes/base_link.stl scale=0.001 0.001 0.001
- added link wheel_arm_leftfront, mass 0.34336062020263136; collision mesh filename=package://patasmonkey_description/meshes/wheel_arm.stl scale=0.001 0.001 0.001; visual mesh filename=package://patasmonkey_description/meshes/wheel_arm.stl scale=0.001 0.001 0.001
- added link wheel_arm_leftrear, mass 0.34336062020263136; collision mesh filename=package://patasmonkey_description/meshes/wheel_arm.stl scale=0.001 0.001 0.001; visual mesh filename=package://patasmonkey_description/meshes/wheel_arm.stl scale=0.001 0.001 0.001
- added link wheel_arm_rightfront, mass 0.34336062020263136; collision mesh filename=package://patasmonkey_description/meshes/wheel_arm.stl scale=0.001 0.001 0.001; visual mesh filename=package://patasmonkey_description/meshes/wheel_arm.stl scale=0.001 0.001 0.001
- added link wheel_arm_rightrear, mass 0.34336062020263136; collision mesh filename=package://patasmonkey_description/meshes/wheel_arm.stl scale=0.001 0.001 0.001; visual mesh filename=package://patasmonkey_description/meshes/wheel_arm.stl scale=0.001 0.001 0.001
- added link wheel_leftfront, mass 0.6459736269326636; collision mesh filename=package://patasmonkey_description/meshes/wheel.stl scale=0.001 0.001 0.001; visual mesh filename=package://patasmonkey_description/meshes/wheel.stl scale=0.001 0.001 0.001
- added link wheel_leftrear, mass 0.6459736269326636; collision mesh filename=package://patasmonkey_description/meshes/wheel.stl scale=0.001 0.001 0.001; visual mesh filename=package://patasmonkey_description/meshes/wheel.stl scale=0.001 0.001 0.001
- added link wheel_rightfront, mass 0.6459736269326636; collision mesh filename=package://patasmonkey_description/meshes/wheel.stl scale=0.001 0.001 0.001; visual mesh filename=package://patasmonkey_description/meshes/wheel.stl scale=0.001 0.001 0.001
- added link wheel_rightrear, mass 0.6459736269326636; collision mesh filename=package://patasmonkey_description/meshes/wheel.stl scale=0.001 0.001 0.001; visual mesh filename=package://patasmonkey_description/meshes/wheel.stl scale=0.001 0.001 0.001
Joints:
- joint rev0: child wheel_arm_v6:1 -> wheel_arm_leftfront; parent base_link_v4:1 -> base_link
- joint rev1: child wheel_arm_v6:2 -> wheel_arm_leftrear; parent base_link_v4:1 -> base_link
- joint rev2: child wheel_arm_v6:3 -> wheel_arm_rightrear; parent base_link_v4:1 -> base_link
- joint rev3: child wheel_arm_v6:4 -> wheel_arm_rightfront; parent base_link_v4:1 -> base_link
- joint rev4: child wheel_v2:1 -> wheel_leftfront; parent wheel_arm_v6:1 -> wheel_arm_leftfront
- joint rev5: child wheel_v2:2 -> wheel_leftrear; parent wheel_arm_v6:2 -> wheel_arm_leftrear
- joint rev6: child wheel_v2:3 -> wheel_rightrear; parent wheel_arm_v6:3 -> wheel_arm_rightrear
- joint rev7: child wheel_v2:4 -> wheel_rightfront; parent wheel_arm_v6:4 -> wheel_arm_rightfront

Commit message: update robot description

File: src/patasmonkey_description/urdf/patasmonkey.urdf (robot description, URDF)
Before this commit: robot patasmonkey_ugv, 9 links, 8 joints
Links:
- removed link wheel_arm_leftfront
- removed link wheel_arm_leftrear
- removed link wheel_arm_rightfront
- removed link wheel_arm_rightrear
- removed link wheel_leftfront
- removed link wheel_leftrear
- removed link wheel_rightfront
- removed link wheel_rightrear
- added link body, mass 8.878175441817634; collision mesh filename=package://patasmonkey_description/meshes/body.stl scale=0.001 0.001 0.001; visual mesh filename=package://patasmonkey_description/meshes/body.stl scale=0.001 0.001 0.001
- added link wheel_v1:1, mass 0.6459736269326636; collision mesh filename=package://patasmonkey_description/meshes/wheel_v1.stl scale=0.001 0.001 0.001; visual mesh filename=package://patasmonkey_description/meshes/wheel_v1.stl scale=0.001 0.001 0.001
- added link wheel_v1:2, mass 0.6459736269326636; collision mesh filename=package://patasmonkey_description/meshes/wheel_v1.stl scale=0.001 0.001 0.001; visual mesh filename=package://patasmonkey_description/meshes/wheel_v1.stl scale=0.001 0.001 0.001
- added link wheel_v1:3, mass 0.6459736269326636; collision mesh filename=package://patasmonkey_description/meshes/wheel_v1.stl scale=0.001 0.001 0.001; visual mesh filename=package://patasmonkey_description/meshes/wheel_v1.stl scale=0.001 0.001 0.001
- added link wheel_v1:4, mass 0.6459736269326636; collision mesh filename=package://patasmonkey_description/meshes/wheel_v1.stl scale=0.001 0.001 0.001; visual mesh filename=package://patasmonkey_description/meshes/wheel_v1.stl scale=0.001 0.001 0.001
- added link wheelarm_1_v3:1, mass 0.11129201234266223; collision mesh filename=package://patasmonkey_description/meshes/wheelarm_1_v3.stl scale=0.001 0.001 0.001; visual mesh filename=package://patasmonkey_description/meshes/wheelarm_1_v3.stl scale=0.001 0.001 0.001
- added link wheelarm_1_v3:2, mass 0.11129201234266223; collision mesh filename=package://patasmonkey_description/meshes/wheelarm_1_v3.stl scale=0.001 0.001 0.001; visual mesh filename=package://patasmonkey_description/meshes/wheelarm_1_v3.stl scale=0.001 0.001 0.001
- added link wheelarm_2_v4:1, mass 0.1112920123426623; collision mesh filename=package://patasmonkey_description/meshes/wheelarm_2_v4.stl scale=0.001 0.001 0.001; visual mesh filename=package://patasmonkey_description/meshes/wheelarm_2_v4.stl scale=0.001 0.001 0.001
- added link wheelarm_2_v4:2, mass 0.1112920123426623; collision mesh filename=package://patasmonkey_description/meshes/wheelarm_2_v4.stl scale=0.001 0.001 0.001; visual mesh filename=package://patasmonkey_description/meshes/wheelarm_2_v4.stl scale=0.001 0.001 0.001
- link base_link: mass 8.831101767270535 -> None; geometry 
Joints:
- added joint base_link_to_body: type fixed, parent base_link, child body, origin xyz=0 0 0 rpy=0 0 -1.57079632679
- joint rev0: child wheel_arm_leftfront -> wheelarm_1_v3:1; origin xyz=0.09999999999999998 -0.030000000000000006 0.05000000000000001 rpy=0 0 0 -> xyz=0.11999999999999998 -7.50720839698537e-18 0.10000000000000002 rpy=0 0 0; parent base_link -> body
- joint rev1: child wheel_arm_leftrear -> wheelarm_2_v4:1; origin xyz=0.09999999999999998 0.03 0.05 rpy=0 0 0 -> xyz=0.13 4.440892098500626e-18 0.10000000000000002 rpy=0 0 0; parent base_link -> body
- joint rev2: child wheel_arm_rightrear -> wheelarm_1_v3:2; origin xyz=-0.1 0.03 0.05 rpy=0 0 0 -> xyz=-0.12 0.0 0.1 rpy=0 0 0; parent base_link -> body
- joint rev3: child wheel_arm_rightfront -> wheelarm_2_v4:2; origin xyz=-0.10000000000000002 -0.030000000000000006 0.05000000000000001 rpy=0 0 0 -> xyz=-0.13 0.0 0.1 rpy=0 0 0; parent base_link -> body
- joint rev4: axis 1.0 0.0 0.0 -> -1.0000000000000064 0.0 0.0; child wheel_leftfront -> wheel_v1:1; origin xyz=0.05000000000000002 -0.15035081932574534 -0.05472322293210703 rpy=0 0 0 -> xyz=0.048000000000000306 -0.16012172781242637 -0.10004368005208156 rpy=0 0 0; parent wheel_arm_leftfront -> wheelarm_1_v3:1
- joint rev5: axis 1.0 0.0 0.0 -> -1.0000000000000009 0.0 0.0; child wheel_leftrear -> wheel_v1:2; origin xyz=0.05000000000000002 0.15035081932574534 -0.054723222932107 rpy=0 0 0 -> xyz=0.03800000000000012 0.16012172781242617 -0.10004368005208177 rpy=0 0 0; parent wheel_arm_leftrear -> wheelarm_2_v4:1
- joint rev6: child wheel_rightrear -> wheel_v1:3; origin xyz=-0.04999999999999999 0.15035081932574534 -0.054723222932107 rpy=0 0 0 -> xyz=-0.04800000000000004 0.16012172781242623 -0.10004368005208186 rpy=0 0 0; parent wheel_arm_rightrear -> wheelarm_1_v3:2
- joint rev7: child wheel_rightfront -> wheel_v1:4; origin xyz=-0.05 -0.15035081932574534 -0.05472322293210703 rpy=0 0 0 -> xyz=-0.038000000000000006 -0.16012172781242623 -0.10004368005208186 rpy=0 0 0; parent wheel_arm_rightfront -> wheelarm_2_v4:2
