Commit message: renamed joints and axes

File: src/patasmonkey_description/urdf/patasmonkey.urdf (robot description, URDF)
Before this commit: robot patasmonkey, 10 links, 9 joints
Links:
- removed link wheel_v1:1
- removed link wheel_v1:2
- removed link wheel_v1:3
- removed link wheel_v1:4
- removed link wheelarm_1_v3:1
- removed link wheelarm_1_v3:2
- removed link wheelarm_2_v4:1
- removed link wheelarm_2_v4:2
- added link wheel_leftfront, mass 0.6459736269326636; collision mesh filename=package://patasmonkey_description/meshes/wheel.stl scale=0.001 0.001 0.001; visual mesh filename=package://patasmonkey_description/meshes/wheel.stl scale=0.001 0.001 0.001
- added link wheel_leftrear, mass 0.6459736269326636; collision mesh filename=package://patasmonkey_description/meshes/wheel.stl scale=0.001 0.001 0.001; visual mesh filename=package://patasmonkey_description/meshes/wheel.stl scale=0.001 0.001 0.001
- added link wheel_rightfront, mass 0.6459736269326636; collision mesh filename=package://patasmonkey_description/meshes/wheel.stl scale=0.001 0.001 0.001; visual mesh filename=package://patasmonkey_description/meshes/wheel.stl scale=0.001 0.001 0.001
- added link wheel_rightrear, mass 0.6459736269326636; collision mesh filename=package://patasmonkey_description/meshes/wheel.stl scale=0.001 0.001 0.001; visual mesh filename=package://patasmonkey_description/meshes/wheel.stl scale=0.001 0.001 0.001
- added link wheelarm_leftfront, mass 0.11129201234266223; collision mesh filename=package://patasmonkey_description/meshes/wheelarm_1.stl scale=0.001 0.001 0.001; visual mesh filename=package://patasmonkey_description/meshes/wheelarm_1.stl scale=0.001 0.001 0.001
- added link wheelarm_leftrear, mass 0.1112920123426623; collision mesh filename=package://patasmonkey_description/meshes/wheelarm_2.stl scale=0.001 0.001 0.001; visual mesh filename=package://patasmonkey_description/meshes/wheelarm_2.stl scale=0.001 0.001 0.001
- added link wheelarm_rightfront, mass 0.1112920123426623; collision mesh filename=package://patasmonkey_description/meshes/wheelarm_2.stl scale=0.001 0.001 0.001; visual mesh filename=package://patasmonkey_description/meshes/wheelarm_2.stl scale=0.001 0.001 0.001
- added link wheelarm_rightrear, mass 0.11129201234266223; collision mesh filename=package://patasmonkey_description/meshes/wheelarm_1.stl scale=0.001 0.001 0.001; visual mesh filename=package://patasmonkey_description/meshes/wheelarm_1.stl scale=0.001 0.001 0.001
Joints:
- removed joint rev0
- removed joint rev1
- removed joint rev2
- removed joint rev3
- removed joint rev4
- removed joint rev5
- removed joint rev6
- removed joint rev7
- added joint wheelarmjoint_leftfront: type continuous, parent body, child wheelarm_leftfront, origin xyz=-0.12 0.0 0.1 rpy=0 0 0, axis 1.0 0.0 0.0
- added joint wheelarmjoint_leftrear: type continuous, parent body, child wheelarm_leftrear, origin xyz=-0.13 0.0 0.1 rpy=0 0 0, axis 1.0 0.0 0.0
- added joint wheelarmjoint_rightfront: type continuous, parent body, child wheelarm_rightfront, origin xyz=0.13 4.440892098500626e-18 0.10000000000000002 rpy=0 0 0, axis -1.0 0.0 0.0
- added joint wheelarmjoint_rightrear: type continuous, parent body, child wheelarm_rightrear, origin xyz=0.11999999999999998 -7.50720839698537e-18 0.10000000000000002 rpy=0 0 0, axis -1.0 0.0 0.0
- added joint wheelaxis_leftfront: type continuous, parent wheelarm_leftfront, child wheel_leftfront, origin xyz=-0.04800000000000004 0.16012172781242623 -0.10004368005208186 rpy=0 0 0, axis 1.0 0.0 0.0
- added joint wheelaxis_leftrear: type continuous, parent wheelarm_leftrear, child wheel_leftrear, origin xyz=-0.038000000000000006 -0.16012172781242623 -0.10004368005208186 rpy=0 0 0, axis 1.0 0.0 0.0
- added joint wheelaxis_rightfromt: type continuous, parent wheelarm_rightfront, child wheel_rightfront, origin xyz=0.03800000000000012 0.16012172781242617 -0.10004368005208177 rpy=0 0 0, axis -1.0000000000000009 0.0 0.0
- added joint wheelaxis_rightrear: type continuous, parent wheelarm_rightrear, child wheel_rightrear, origin xyz=0.048000000000000306 -0.16012172781242637 -0.10004368005208156 rpy=0 0 0, axis -1.0000000000000064 0.0 0.0

Commit message: visualized wheel odometry and robot model motion in rviz

File: src/patasmonkey_description/urdf/patasmonkey.urdf (robot description, URDF)
Before this commit: robot patasmonkey, 10 links, 9 joints
Joints:
- removed joint wheelaxis_rightfromt
- added joint wheelaxis_rightfront: type continuous, parent wheelarm_rightfront, child wheel_rightfront, origin xyz=0.03800000000000012 0.16012172781242617 -0.10004368005208177 rpy=0 0 0, axis -1.0 0.0 0.0
- joint wheelaxis_leftfront: axis 1.0 0.0 0.0 -> -1.0 0.0 0.0
- joint wheelaxis_leftrear: axis 1.0 0.0 0.0 -> -1.0 0.0 0.0
- joint wheelaxis_rightrear: axis -1.0000000000000064 0.0 0.0 -> -1.0 0.0 0.0
