Commit message: add imu_link to urdf file

File: src/pm_description/urdf/pm.urdf (robot description, URDF)
Before this commit: robot patasmonkey, 10 links, 9 joints
Links:
- added link imu_link; visual box size=0.04 0.04 0.015
Joints:
- added joint base_link_to_imu_link: type fixed, parent base_link, child imu_link, origin xyz=0.0 0.0 0.01 rpy=0.0 0.0 0.0

Commit message: update package name for meshes

File: src/pm_description/urdf/pm.urdf (robot description, URDF)
Before this commit: robot patasmonkey, 11 links, 10 joints
Links:
- link body: geometry collision mesh filename=package://pm_description/meshes/body.stl scale=0.001 0.001 0.001; visual mesh filename=package://pm_description/meshes/body.stl scale=0.001 0.001 0.001
- link wheel_leftfront: geometry collision mesh filename=package://pm_description/meshes/wheel.stl scale=0.001 0.001 0.001; visual mesh filename=package://pm_description/meshes/wheel.stl scale=0.001 0.001 0.001
- link wheel_leftrear: geometry collision mesh filename=package://pm_description/meshes/wheel.stl scale=0.001 0.001 0.001; visual mesh filename=package://pm_description/meshes/wheel.stl scale=0.001 0.001 0.001
- link wheel_rightfront: geometry collision mesh filename=package://pm_description/meshes/wheel.stl scale=0.001 0.001 0.001; visual mesh filename=package://pm_description/meshes/wheel.stl scale=0.001 0.001 0.001
- link wheel_rightrear: geometry collision mesh filename=package://pm_description/meshes/wheel.stl scale=0.001 0.001 0.001; visual mesh filename=package://pm_description/meshes/wheel.stl scale=0.001 0.001 0.001
- link wheelarm_leftfront: geometry collision mesh filename=package://pm_description/meshes/wheelarm_1.stl scale=0.001 0.001 0.001; visual mesh filename=package://pm_description/meshes/wheelarm_1.stl scale=0.001 0.001 0.001
- link wheelarm_leftrear: geometry collision mesh filename=package://pm_description/meshes/wheelarm_2.stl scale=0.001 0.001 0.001; visual mesh filename=package://pm_description/meshes/wheelarm_2.stl scale=0.001 0.001 0.001
- link wheelarm_rightfront: geometry collision mesh filename=package://pm_description/meshes/wheelarm_2.stl scale=0.001 0.001 0.001; visual mesh filename=package://pm_description/meshes/wheelarm_2.stl scale=0.001 0.001 0.001
- link wheelarm_rightrear: geometry collision mesh filename=package://pm_description/meshes/wheelarm_1.stl scale=0.001 0.001 0.001; visual mesh filename=package://pm_description/meshes/wheelarm_1.stl scale=0.001 0.001 0.001

Commit message: adjusted imu orientation

File: src/pm_description/urdf/pm.urdf (robot description, URDF)
Before this commit: robot patasmonkey, 11 links, 10 joints
Joints:
- joint base_link_to_imu_link: origin xyz=0.0 0.0 0.01 rpy=0.0 0.0 0.0 -> xyz=0.0 0.0 0.01 rpy=0.0 0.0 -1.5708

Commit message: update axes to adjust to ROS coordinates

File: src/pm_description/urdf/pm.urdf (robot description, URDF)
Before this commit: robot patasmonkey, 11 links, 10 joints
Joints:
- joint base_link_to_imu_link: origin xyz=0.0 0.0 0.01 rpy=0.0 0.0 -1.5708 -> xyz=0.0 0.0 0.01 rpy=0.0 0.0 0.0

Commit message: add camera related links to urdf file

File: src/pm_description/urdf/pm.urdf (robot description, URDF)
Before this commit: robot patasmonkey, 11 links, 10 joints
Links:
- added link cam0_link
- added link cam0_optical_frame
- added link cam1_link
- added link cam1_optical_frame
- added link oakd_imu_link
- added link oakd_link; visual box size=0.09 0.03 0.025
- added link rgb_camera_link
- added link rgb_camera_optical_frame
Joints:
- added joint base_link_to_oakd_link: type fixed, parent base_link, child oakd_link, origin xyz=0.0 0.0 0.28 rpy=0.0 0.0 0.0
- added joint cam0_link_to_cam0_optical_frame: type fixed, parent cam0_link, child cam0_optical_frame, origin xyz=0.0 0.0 0.0 rpy=-1.57079632679 0.0 -1.57079632679
- added joint cam1_link_to_cam1_optical_frame: type fixed, parent cam1_link, child cam1_optical_frame, origin xyz=0.0 0.0 0.0 rpy=-1.57079632679 0.0 -1.57079632679
- added joint oakd_link_to_cam0_link: type fixed, parent oakd_link, child cam0_link, origin xyz=0.0 0.0376655 0.0 rpy=0.0 0.0 0.0
- added joint oakd_link_to_cam1_link: type fixed, parent oakd_link, child cam1_link, origin xyz=0.0 -0.0376655 0.0 rpy=0.0 0.0 0.0
- added joint oakd_link_to_oakd_imu_link: type fixed, parent oakd_link, child oakd_imu_link, origin xyz=0.0 0.0 0.0 rpy=0.0 0.0 0.0
- added joint oakd_link_to_rgb_camera_link: type fixed, parent oakd_link, child rgb_camera_link, origin xyz=0.0 0.0 0.0 rpy=0.0 0.0 0.0
- added joint rgb_camera_link_to_rgb_camera_optical_frame: type fixed, parent rgb_camera_link, child rgb_camera_optical_frame, origin xyz=0.0 0.0 0.0 rpy=-1.57079632679 0.0 -1.57079632679

Commit message: updated localization affairs

File: src/pm_description/urdf/pm.urdf (robot description, URDF)
Before this commit: robot patasmonkey, 19 links, 18 joints
Links:
- added link gps_link
Joints:
- added joint gps_joint: type fixed, parent base_link, child gps_link, origin xyz=-0.02 -0.07 0.25 rpy=0 0 0

Commit message: update link name of HWT905 IMU

File: src/pm_description/urdf/pm.urdf (robot description, URDF)
Before this commit: robot patasmonkey, 20 links, 19 joints
Links:
- removed link imu_link
- added link wit_imu_link; visual box size=0.04 0.04 0.015
Joints:
- removed joint base_link_to_imu_link
- added joint base_link_to_wit_imu_link: type fixed, parent base_link, child wit_imu_link, origin xyz=0.0 0.0 0.01 rpy=0.0 0.0 0.0

Commit message: checking visual odometry output

File: src/pm_description/urdf/pm.urdf (robot description, URDF)
Before this commit: robot patasmonkey, 20 links, 19 joints
Joints:
- joint oakd_link_to_oakd_imu_link: origin xyz=0.0 0.0 0.0 rpy=0.0 0.0 0.0 -> xyz=0.0 0.0 0.0 rpy=1.57079632679 0.0 1.57079632679

Commit message: checking visual odometry output

File: src/pm_description/urdf/pm.urdf (robot description, URDF)
Before this commit: robot patasmonkey, 20 links, 19 joints
Joints:
- joint oakd_link_to_oakd_imu_link: origin xyz=0.0 0.0 0.0 rpy=1.57079632679 0.0 1.57079632679 -> xyz=0.0 0.0 0.0 rpy=-1.57079632679 0.0 1.57079632679

Commit message: rotated joint from  oak-d to oak-d-imu

File: src/pm_description/urdf/pm.urdf (robot description, URDF)
Before this commit: robot patasmonkey, 20 links, 19 joints
Joints:
- joint oakd_link_to_oakd_imu_link: origin xyz=0.0 0.0 0.0 rpy=-1.57079632679 0.0 1.57079632679 -> xyz=0.0 0.0 0.0 rpy=0.0 0.0 0.0

Commit message: add diagnostics function to adapt TF from VO to PM

File: src/pm_description/urdf/pm.urdf (robot description, URDF)
Before this commit: robot patasmonkey, 20 links, 19 joints
Links:
- added link openvins_imu_link
Joints:
- added joint oakd_link_to_openvins_imu_link: type fixed, parent oakd_link, child openvins_imu_link, origin xyz=0.0 0.0 0.0 rpy=0.0 0.0 0.0

Commit message: adjust joint rpy for VO

File: src/pm_description/urdf/pm.urdf (robot description, URDF)
Before this commit: robot patasmonkey, 21 links, 20 joints
Joints:
- joint oakd_link_to_openvins_imu_link: origin xyz=0.0 0.0 0.0 rpy=0.0 0.0 0.0 -> xyz=0.0 0.0 0.0 rpy=-1.57079632679 0.0 1.57079632679

Commit message: adjust joint rpy and adapter node for VO

File: src/pm_description/urdf/pm.urdf (robot description, URDF)
Before this commit: robot patasmonkey, 21 links, 20 joints
Joints:
- joint oakd_link_to_openvins_imu_link: origin xyz=0.0 0.0 0.0 rpy=-1.57079632679 0.0 1.57079632679 -> xyz=0.0 0.0 0.0 rpy=0.0 0.0 0.0
